File: kicad_poc.kicad_pcb (KiCad board)
At the start: 2 copper layers, 394.6 x 252.4 mm, 61 parts

Commit message: working state - imported pcb and outline, before doing routes
Parts:
- S1, S10, S11, S12, S13, S14, S15, S16, S17, S18, S19, S2, S20, S21, S22, S23, S24, S25, S26, S27, S28, S29, S3, S30, S4, S5, S6, S7, S8, S9: footprint ceoloide:switch_mx -> MX; moved to F.Cu
- moved D1 11.6 mm to (24.0, 78.4), turned to 169 degrees
- moved D10 11.6 mm to (82.2, 78.0), turned to 169 degrees
- moved D12 11.6 mm to (97.2, 100.3), turned to 169 degrees
- moved D16 11.6 mm to (272.8, 78.4), turned to -169 degrees
- moved D19 11.6 mm to (251.7, 69.8), turned to -169 degrees
- moved D21 11.6 mm to (235.5, 85.9), turned to -169 degrees
- moved D22 11.6 mm to (231.9, 67.2), turned to -169 degrees
- moved D23 11.6 mm to (228.3, 48.6), turned to -169 degrees
- moved D24 11.6 mm to (218.3, 96.7), turned to -169 degrees
- moved D25 11.6 mm to (214.6, 78.0), turned to -169 degrees
- moved D27 11.6 mm to (199.6, 100.3), turned to -169 degrees
- moved D4 11.6 mm to (45.1, 69.8), turned to 169 degrees
- moved D6 11.6 mm to (61.3, 85.9), turned to 169 degrees
- moved D7 11.6 mm to (64.9, 67.2), turned to 169 degrees
- moved D8 11.6 mm to (68.5, 48.6), turned to 169 degrees
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Connections:
- S1 pad 1: P14 -> pinky_home
- S1 pad 2: pinky_home -> P14
- S10 pad 1: P7 -> index_home
- S10 pad 2: index_home -> P7
- S11 pad 1: P7 -> index_top
- S11 pad 2: index_top -> P7
- S12 pad 1: P8 -> inner_bottom
- S12 pad 2: inner_bottom -> P8
- S13 pad 1: P8 -> inner_home
- S13 pad 2: inner_home -> P8
- S14 pad 1: P8 -> inner_top
- S14 pad 2: inner_top -> P8
- S15 pad 1: P14 -> center_single
- S15 pad 2: center_single -> P14
- S16 pad 1: P14 -> mirror_pinky_home
- S16 pad 2: mirror_pinky_home -> P14
- S17 pad 1: P14 -> mirror_pinky_top
- S17 pad 2: mirror_pinky_top -> P14
- S18 pad 1: P16 -> mirror_ring_bottom
- S18 pad 2: mirror_ring_bottom -> P16
- S19 pad 1: P16 -> mirror_ring_home
- S19 pad 2: mirror_ring_home -> P16
- S2 pad 1: P14 -> pinky_top
- S2 pad 2: pinky_top -> P14
- S20 pad 1: P16 -> mirror_ring_top
- S20 pad 2: mirror_ring_top -> P16
- S21 pad 1: P10 -> mirror_middle_bottom
- S21 pad 2: mirror_middle_bottom -> P10
- S22 pad 1: P10 -> mirror_middle_home
- S22 pad 2: mirror_middle_home -> P10
- S23 pad 1: P10 -> mirror_middle_top
- S23 pad 2: mirror_middle_top -> P10
- S24 pad 1: P7 -> mirror_index_bottom
- S24 pad 2: mirror_index_bottom -> P7
- S25 pad 1: P7 -> mirror_index_home
- S25 pad 2: mirror_index_home -> P7
- S26 pad 1: P7 -> mirror_index_top
- S26 pad 2: mirror_index_top -> P7
- S27 pad 1: P8 -> mirror_inner_bottom
- S27 pad 2: mirror_inner_bottom -> P8
- S28 pad 1: P8 -> mirror_inner_home
- S28 pad 2: mirror_inner_home -> P8
- S29 pad 1: P8 -> mirror_inner_top
- S29 pad 2: mirror_inner_top -> P8
- S3 pad 1: P16 -> ring_bottom
- S3 pad 2: ring_bottom -> P16
- S30 pad 1: P14 -> mirror_center_single
- S30 pad 2: mirror_center_single -> P14
- S4 pad 1: P16 -> ring_home
- S4 pad 2: ring_home -> P16
- S5 pad 1: P16 -> ring_top
- S5 pad 2: ring_top -> P16
- S6 pad 1: P10 -> middle_bottom
- S6 pad 2: middle_bottom -> P10
- S7 pad 1: P10 -> middle_home
- S7 pad 2: middle_home -> P10
- S8 pad 1: P10 -> middle_top
- S8 pad 2: middle_top -> P10
- S9 pad 1: P7 -> index_bottom
- S9 pad 2: index_bottom -> P7
Other:
- board size 394.6 x 252.4 mm -> 268.2 x 113 mm

Commit message: added simple single side routings on both sides
Parts:
- moved D16 24.4 mm to (271.2, 102.8), turned to 180 degrees
- moved S16 24.3 mm to (271.2, 97.8), turned to 0 degrees
- moved S17 24.1 mm to (271.2, 78.8), turned to 0 degrees
- moved D17 24.1 mm to (271.2, 83.8), turned to 180 degrees
- moved D1 23.3 mm to (27.0, 55.3), turned to 158 degrees
- moved S1 23.2 mm to (28.8, 50.7), turned to -22 degrees
- moved S2 23.0 mm to (36.0, 33.1), turned to -22 degrees
- moved D2 23.0 mm to (34.1, 37.7), turned to 158 degrees
- moved D18 21.1 mm to (252.2, 109.3), turned to 180 degrees
- moved S18 20.9 mm to (252.2, 104.3), turned to 0 degrees
- moved S20 20.7 mm to (252.2, 66.3), turned to 0 degrees
- moved D20 20.6 mm to (252.2, 71.3), turned to 180 degrees
- moved D19 20.5 mm to (252.2, 90.3), turned to 180 degrees
- moved S19 20.5 mm to (252.2, 85.3), turned to 0 degrees
- moved D3 20.0 mm to (42.1, 68.5), turned to 158 degrees
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Routing:
- net P16: track 0.00 -> 114.2 mm
- net P7: track 0.00 -> 114.2 mm
- net P10: track 0.00 -> 96.5 mm
- net P8: track 0.00 -> 77.6 mm
- net P14: track 0.00 -> 40.2 mm
- net mirror_pinky_home: track 0.00 -> 11.5 mm
- net mirror_inner_top: track 0.00 -> 10.2 mm
- net mirror_middle_bottom: track 0.00 -> 10.2 mm
- net mirror_inner_bottom: track 0.00 -> 10.2 mm
- net pinky_top: track 0.00 -> 10.2 mm
- net inner_top: track 0.00 -> 10.2 mm
- net middle_home: track 0.00 -> 10.2 mm
- net inner_bottom: track 0.00 -> 10.2 mm
- net mirror_ring_top: track 0.00 -> 10.2 mm
- net mirror_ring_home: track 0.00 -> 10.2 mm
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Other:
- board size 268.2 x 113 mm -> 263.4 x 138.9 mm

Commit message: latest with a working dxf
Parts:
- moved D1 24.1 mm to (23.2, 79.1), turned to 169 degrees
- moved S1 24.0 mm to (24.2, 74.2), turned to -11 degrees
- moved S2 23.9 mm to (27.8, 55.5), turned to -11 degrees
- moved D2 23.9 mm to (26.9, 60.4), turned to 169 degrees
- moved D16 23.7 mm to (272.0, 79.1), turned to -169 degrees
- moved S16 23.6 mm to (271.0, 74.2), turned to 11 degrees
- moved S17 23.5 mm to (267.4, 55.5), turned to 11 degrees
- moved D17 23.5 mm to (268.4, 60.4), turned to -169 degrees
- moved D3 20.7 mm to (40.7, 89.1), turned to 169 degrees
- moved S5 20.6 mm to (48.9, 46.9), turned to -11 degrees
- moved S3 20.5 mm to (41.6, 84.2), turned to -11 degrees
- moved D5 20.4 mm to (47.9, 51.8), turned to 169 degrees
- moved D18 20.3 mm to (254.6, 89.1), turned to -169 degrees
- moved S20 20.2 mm to (246.4, 46.9), turned to 11 degrees
- moved D4 20.2 mm to (44.3, 70.4), turned to 169 degrees
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Other:
- board size 263.4 x 138.9 mm -> 268.2 x 113 mm

Commit message: each side routed
Parts:
- moved D16 24.4 mm to (270.4, 103.4), turned to 180 degrees
- moved S16 24.3 mm to (270.4, 98.4), turned to 0 degrees
- moved S17 24.1 mm to (270.4, 79.4), turned to 0 degrees
- moved D17 24.1 mm to (270.4, 84.4), turned to 180 degrees
- moved D1 23.3 mm to (26.2, 56.0), turned to 158 degrees
- moved S1 23.2 mm to (28.1, 51.3), turned to -22 degrees
- moved S2 23.0 mm to (35.2, 33.7), turned to -22 degrees
- moved D2 23.0 mm to (33.3, 38.4), turned to 158 degrees
- moved D18 21.1 mm to (251.4, 109.9), turned to 180 degrees
- moved S18 20.9 mm to (251.4, 104.9), turned to 0 degrees
- moved S20 20.7 mm to (251.4, 66.9), turned to 0 degrees
- moved D20 20.6 mm to (251.4, 71.9), turned to 180 degrees
- moved D19 20.5 mm to (251.4, 90.9), turned to 180 degrees
- moved S19 20.5 mm to (251.4, 85.9), turned to 0 degrees
- moved D3 20.0 mm to (41.4, 69.1), turned to 158 degrees
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Routing:
- net P14: track 40.2 -> 242.5 mm, vias 0 -> 4
- net P16: track 114.2 -> 280.0 mm, vias 0 -> 4
- net P18: track 0.00 -> 142.1 mm, vias 0 -> 8
- net P6: track 0.00 -> 135.1 mm
- net P15: track 0.00 -> 134.1 mm
- net P19: track 0.00 -> 130.0 mm, vias 0 -> 8
- net P5: track 0.00 -> 127.2 mm, vias 0 -> 10
- net P10: track 96.5 -> 218.6 mm, vias 0 -> 2
- net P4: track 0.00 -> 117.7 mm, vias 0 -> 8
- net P7: track 114.2 -> 214.5 mm, vias 0 -> 4
- net P8: track 77.6 -> 150.0 mm, vias 0 -> 3
- net center_single: track 0.00 -> 10.5 mm
- net mirror_center_single: track 0.00 -> 10.1 mm
- net ring_bottom: track 0.00 -> 9.87 mm
Other:
- board size 268.2 x 113 mm -> 263.4 x 138.9 mm

Commit message: all pcb wiring done!
Parts:
- moved D1 47.9 mm to (25.9, 103.9), turned to 180 degrees
- moved S1 47.6 mm to (25.9, 98.9), turned to 0 degrees
- moved D2 47.1 mm to (25.9, 84.9), turned to 180 degrees
- moved S2 47.1 mm to (25.9, 79.9), turned to 0 degrees
- moved D16 47.0 mm to (270.1, 56.5), turned to -158 degrees
- moved S16 46.7 mm to (268.2, 51.8), turned to 22 degrees
- moved D17 46.2 mm to (263.0, 38.8), turned to -158 degrees
- moved S17 46.2 mm to (261.1, 34.2), turned to 22 degrees
- moved D3 41.4 mm to (44.9, 110.4), turned to 180 degrees
- moved S3 41.0 mm to (44.9, 105.4), turned to 0 degrees
- moved D18 40.5 mm to (254.9, 69.6), turned to -158 degrees
- moved S5 40.2 mm to (44.9, 67.4), turned to 0 degrees
- moved D4 40.1 mm to (44.9, 91.4), turned to 180 degrees
- moved S18 40.0 mm to (253.0, 65.0), turned to 22 degrees
- moved D5 40.0 mm to (44.9, 72.4), turned to 180 degrees
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Routing:
- net P14: track 242.5 -> 718.0 mm, vias 4 -> 9
- net P16: track 280.0 -> 654.8 mm, vias 4 -> 5
- net P7: track 214.5 -> 584.5 mm, vias 4 -> 5
- net P8: track 150.0 -> 519.0 mm
- net P10: track 218.6 -> 584.8 mm, vias 2 -> 3
- net P6: track 135.1 -> 388.0 mm, vias 0 -> 1
- net P15: track 134.1 -> 370.4 mm, vias 0 -> 2
- net P4: track 117.7 -> 329.4 mm, vias 8 -> 10
- net P5: track 127.2 -> 337.1 mm, vias 10 -> 11
- net P18: track 142.1 -> 337.8 mm, vias 8 -> 9
- net P19: track 130.0 -> 313.8 mm, vias 8 -> 14
- net GND: track 0.00 -> 0.69 mm
Other:
- outline, holes or cut-outs redrawn

Commit message: latest - sent to the jlc
Routing:
- net GND: track 0.69 -> 19.4 mm
- added copper zone on B.Cu, net (none)
- added copper zone on F.Cu, net (none)
Changed lines of the file:
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@@
+	)
+	(segment
+		(start 149.793296 83.501795)
+		(end 155.194558 78.100533)
+		(width 0.2)
+		(layer "F.Cu")
+		(net 49)
+	)
+	(segment
+		(start 140.719215 83.501795)
+		(end 140.719215 85.510473)
+		(width 0.2)
+		(layer "F.Cu")
+		(net 49)
+	)
+	(segment
+		(start 140.719215 83.501795)
+		(end 149.793296 83.501795)
+		(width 0.2)
+		(layer "F.Cu")
+		(net 49)
 	)
 	(segment
@@
 		(net 52)
 	)
+	(zone
+		(net 0)
+		(net_name "")
+		(layers "F.Cu" "B.Cu")
+		(hatch edge 0.5)
+		(connect_pads
+			(clearance 0.5)
+		)
+		(min_thickness 0.25)
+		(filled_areas_thickness no)
+		(fill yes
+			(thermal_gap 0.5)
+			(thermal_bridge_width 0.5)
+			(island_removal_mode 1)
+			(island_area_min 9.999999)
+		)
+		(polygon
+			(pts
+				(xy -1.778 -5.334) (xy 298.196 -3.048) (xy 301.752 115.824) (xy 230.632 168.656) (xy 53.594 175.768)
+				(xy -11.684 115.824)
+			)
+		)
+	)
 	(group ""
